File: Power Regulation.kicad_sch (KiCad schematic)
At the start: 20 parts, among them Q1 PMOS, SW1 SW_SPST, SW2 SW_SPST, U1 LM1085-ADJ, U8 TPS561243DRLR

Commit message: Added some footprints and made some connections
Parts:
- C1, C2, C26, C27, C28: footprint (none) -> Capacitor_SMD:C_0603_1608Metric
- R1, R10, R11, R12, R13, R14, R2, R9: footprint (none) -> Resistor_SMD:R_0603_1608Metric
- U1: footprint (none) -> Package_TO_SOT_SMD:TO-263-3_TabPin2
Changed lines of the file:
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@@
 			)
 		)
-		(property "Footprint" ""
+		(property "Footprint" "Resistor_SMD:R_0603_1608Metric"
 			(at 96.012 102.87 90)
 			(effects
@@
 			)
 		)
-		(property "Footprint" ""
+		(property "Footprint" "Resistor_SMD:R_0603_1608Metric"
 			(at 84.582 110.49 90)
 			(effects
@@
 			)
 		)
-		(property "Footprint" ""
+		(property "Footprint" "Capacitor_SMD:C_0603_1608Metric"
 			(at 206.7052 107.95 0)
 			(effects
@@
 			)
 		)
-		(property "Footprint" ""
+		(property "Footprint" "Resistor_SMD:R_0603_1608Metric"
 			(at 179.832 113.03 90)
 			(effects
@@
 			)
 		)
-		(property "Footprint" ""
+		(property "Footprint" "Package_TO_SOT_SMD:TO-263-3_TabPin2"
 			(at 219.71 92.71 0)
 			(effects
@@
 			)
 		)
-		(property "Footprint" ""
+		(property "Footprint" "Resistor_SMD:R_0603_1608Metric"
 			(at 124.46 105.918 90)
 			(effects
@@
 			)
 		)
-		(property "Footprint" ""
+		(property "Footprint" "Resistor_SMD:R_0603_1608Metric"
 			(at 179.832 105.41 90)
 			(effects
@@
 			)
 		)
-		(property "Footprint" ""
+		(property "Footprint" "Resistor_SMD:R_0603_1608Metric"
 			(at 96.012 113.03 90)
 			(effects
@@
 			)
 		)
-		(property "Footprint" ""
+		(property "Footprint" "Resistor_SMD:R_0603_1608Metric"
 			(at 226.822 102.87 90)
 			(effects
@@
 			)
 		)
-		(property "Footprint" ""
+		(property "Footprint" "Capacitor_SMD:C_0603_1608Metric"
 			(at 191.4652 107.95 0)
 			(effects
@@
 			)
 		)
-		(property "Footprint" ""
+		(property "Footprint" "Capacitor_SMD:C_0603_1608Metric"
 			(at 112.7252 107.95 0)
 			(effects
@@
 			)
 		)
-		(property "Footprint" ""
+		(property "Footprint" "Capacitor_SMD:C_0603_1608Metric"
 			(at 238.4552 107.95 0)
 			(effects
@@
 			)
 		)
-		(property "Footprint" ""
+		(property "Footprint" "Capacitor_SMD:C_0603_1608Metric"
 			(at 166.37 103.1748 0)
 			(effects
@@
 			)
 		)
-		(property "Footprint" ""
+		(property "Footprint" "Resistor_SMD:R_0603_1608Metric"
 			(at 226.822 110.49 90)
 			(effects

Commit message: initial routing of power and MCU sections
Parts:
- removed L2: L, symbol Device:L
- added C29: 22u, Capacitor_SMD:C_0603_1608Metric, symbol Device:C
- added C30: 0.1u, Capacitor_SMD:C_0603_1608Metric, symbol Device:C
- added L2: IFDC5050HZER270M, Wall_E_footprints:IND_IFDC5050HZER_VIS, symbol Wall_E_parts:IFDC5050HZER270M
- C26: value C -> 2.2u
- C27: value C -> 22u
- F1: footprint (none) -> Fuse:Fuseholder_Blade_Mini_Keystone_3568
- Q1: footprint (none) -> Package_TO_SOT_THT:TO-220-3_Vertical
- SW1, SW2: footprint (none) -> Connector_AMASS:AMASS_XT30PW-F_1x02_P2.50mm_Horizontal
Connections:
- net 5V: now also C29.1, C30.1, L2.1
- net GND: now also C29.2, C30.2
- net buck_sw: now reaches C28.2, U8.2 (SW)
- net buck_sw: now also L2.2
Other:
- moved on the sheet: C1, C2, C27, R1, R12, R13, R2, U1

Commit message: Routing Updates
Parts:
- removed Q1: PMOS, Package_TO_SOT_THT:TO-220-3_Vertical, symbol Simulation_SPICE:PMOS
- added Q1: SI4435FDY-T1-GE3, Wall_E_footprints:SO-8_VIS, symbol Wall_E_parts:SI4435FDY-T1-GE3
Connections:
- net V_in: now also Q1.5, Q1.6, Q1.7, Q1.8
- net at F1.2: now also Q1.1, Q1.2, Q1.3
- net at R9.1: now also Q1.4
Other:
- note added: "Calculations for L: Iout_min = 50mA -> delta I_L = 100mA Vin_max = 13V -> delta V_L = 13-5=8V D = Vin/Vout = 0.385 t = D/f = 0.385/1.28M = 0.3us L = V_L*t/(delta I_L) = 24uH"
- note added: "Thermal Calculations for LDO: Vin = 5V Vout = 3.3V Iout_max = 1A Ploss = (5-3.3)*1 = 1.7W Thermal Resistance = 22.8+15.6 = 38.4 C/W T_rise = 38.4*1.7 = 65.28 T_j = 25+65.28 = 90.28 < T_max = 150C"
- title: (none) -> Wall-E Power Regulation
- moved on the sheet: C1, C2, C26, C27, C28, C29, C30, F1, L2, R1, R10, R11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

Commit message: Final commit before Charlie review
Parts:
- added TP3: TestPoint_Small, TestPoint:TestPoint_Pad_D1.0mm, symbol Connector:TestPoint_Small
- C2, C27, C29: footprint Capacitor_SMD:C_0603_1608Metric -> Capacitor_THT:CP_Radial_D5.0mm_P2.00mm; now not fitted
- F1, SW1, SW2: now not fitted
- R1: value R -> 16.5k 1%
- R2: value R -> 10k 1%
Connections:
- net buck_sw: now also TP3.1
Other:
- moved on the sheet: C1, R1, R2, U1

Commit message: Final design before order
Connections:
- net V_in: now also Q1.1, Q1.2, Q1.3; no longer Q1.5, Q1.6, Q1.7, Q1.8
- new net: F1.2, Q1.5, Q1.6, Q1.7, Q1.8
Other:
- moved on the sheet: Q1, R9
Changed lines of the file:
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@@
+	)
+	(junction
+		(at 63.5 101.6)
+		(diameter 0)
+		(color 0 0 0 0)
 	)
 	(junction
@@
 	)
 	(junction
+		(at 63.5 99.06)
+		(diameter 0)
+		(color 0 0 0 0)
+	)
+	(junction
 		(at 222.25 99.06)
 		(diameter 0)
@@
 	)
 	(junction
-		(at 63.5 97.79)
-		(diameter 0)
-		(color 0 0 0 0)
-	)
-	(junction
 		(at 200.66 99.06)
 		(diameter 0)
@@
 	)
 	(junction
+		(at 93.98 101.6)
+		(diameter 0)
+		(color 0 0 0 0)
+	)
+	(junction
+		(at 257.81 106.68)
+		(diameter 0)
+		(color 0 0 0 0)
+	)
+	(junction
+		(at 104.14 107.95)
+		(diameter 0)
+		(color 0 0 0 0)
+	)
+	(junction
 		(at 93.98 99.06)
 		(diameter 0)
@@
 	)
 	(junction
-		(at 257.81 106.68)
-		(diameter 0)
-		(color 0 0 0 0)
-	)
-	(junction
-		(at 104.14 107.95)
-		(diameter 0)
-		(color 0 0 0 0)
-	)
-	(junction
 		(at 200.66 109.22)
 		(diameter 0)
@@
 	)
 	(junction
-		(at 63.5 99.06)
-		(diameter 0)
-		(color 0 0 0 0)
-	)
-	(junction
-		(at 93.98 97.79)
-		(diameter 0)
-		(color 0 0 0 0)
-	)
-	(junction
 		(at 104.14 99.06)
 		(diameter 0)
@@
 		(color 0 0 0 0)
 	)
-	(junction
-		(at 93.98 100.33)
-		(diameter 0)
-		(color 0 0 0 0)
-	)
 	(wire
 		(pts
@@
 	(wire
 		(pts
-			(xy 93.98 95.25) (xy 93.98 97.79)
+			(xy 93.98 96.52) (xy 97.79 96.52)
+		)
+		(stroke
+			(width 0)
+			(type default)
+		)
+	)
+	(wire
+		(pts
+			(xy 93.98 99.06) (xy 93.98 101.6)
 		)
 		(stroke
@@
 	(wire
 		(pts
-			(xy 93.98 97.79) (xy 93.98 99.06)
+			(xy 63.5 96.52) (xy 63.5 99.06)
 		)
 		(stroke
@@
 	(wire
 		(pts
-			(xy 63.5 113.03) (xy 63.5 110.49)
+			(xy 97.79 87.63) (xy 97.79 88.9)
 		)
 		(stroke
@@
 	(wire
 		(pts
+			(xy 93.98 101.6) (xy 93.98 104.14)
+		)
+		(stroke
+			(width 0)
+			(type default)
+		)
+	)
+	(wire
+		(pts
 			(xy 175.26 92.71) (xy 175.26 99.06)
 		)
@@
 	(wire
 		(pts
-			(xy 63.5 97.79) (xy 63.5 99.06)
-		)
-		(stroke
-			(width 0)
-			(type default)
-		)
-	)
-	(wire
-		(pts
 			(xy 104.14 82.55) (xy 104.14 99.06)
 		)
@@
 	(wire
 		(pts
-			(xy 93.98 100.33) (xy 93.98 102.87)
-		)
-		(stroke
-			(width 0)
-			(type default)
-		)
-	)
-	(wire
-		(pts
 			(xy 104.14 106.68) (xy 104.14 107.95)
 		)
@@
 	(wire
 		(pts
-			(xy 63.5 95.25) (xy 63.5 97.79)
-		)
-		(stroke
-			(width 0)
-			(type default)
-		)
-	)
-	(wire
-		(pts
 			(xy 39.37 99.06) (xy 43.18 99.06)
 		)
@@
 	(wire
 		(pts
+			(xy 63.5 101.6) (xy 63.5 104.14)
+		)
+		(stroke
+			(width 0)
+			(type default)
+		)
+	)
+	(wire
+		(pts
 			(xy 104.14 99.06) (xy 118.11 99.06)
 		)
@@
 	(wire
 		(pts
-			(xy 63.5 99.06) (xy 63.5 100.33)
-		)
-		(stroke
-			(width 0)
-			(type default)
-		)
-	)
-	(wire
-		(pts
 			(xy 175.26 99.06) (xy 176.53 99.06)
 		)
@@
 	(wire
 		(pts
-			(xy 93.98 99.06) (xy 93.98 100.33)
-		)
-		(stroke
-			(width 0)
-			(type default)
-		)
-	)
-	(wire
-		(pts
 			(xy 165.1 114.3) (xy 165.1 116.84)
 		)
@@
 		(pts
 			(xy 238.76 116.84) (xy 238.76 107.95)
+		)
+		(stroke
+			(width 0)
+			(type default)
+		)
+	)
+	(wire
+		(pts
+			(xy 63.5 99.06) (xy 63.5 101.6)
 		)
 		(stroke
@@
 	(symbol
 		(lib_id "power:GND")
-		(at 63.5 113.03 0)
+		(at 97.79 87.63 180)
 		(unit 1)
 		(exclude_from_sim no)
@@
 		(fields_autoplaced yes)
 		(property "Reference" "#PWR036"
-			(at 63.5 119.38 0)
+			(at 97.79 81.28 0)
 			(effects
 				(font
@@
 		)
 		(property "Value" "GND"
-			(at 63.5 118.11 0)
+			(at 97.79 82.55 0)
 			(effects
 				(font
@@
 		)
 		(property "Footprint" ""
-			(at 63.5 113.03 0)
+			(at 97.79 87.63 0)
 			(effects
 				(font
@@
 		)
 		(property "Datasheet" ""
-			(at 63.5 113.03 0)
+			(at 97.79 87.63 0)
 			(effects
 				(font
@@
 		)
 		(property "Description" "Power symbol creates a global label with name \"GND\" , ground"
-			(at 63.5 113.03 0)
+			(at 97.79 87.63 0)
 			(effects
 				(font
@@
 	(symbol
 		(lib_id "Device:R")
-		(at 63.5 106.68 0)
+		(at 97.79 92.71 180)
 		(unit 1)
 		(exclude_from_sim no)
@@
 		(fields_autoplaced yes)
 		(property "Reference" "R9"
-			(at 66.04 105.4099 0)
+			(at 95.25 93.9801 0)
 			(effects
 				(font
@@
 		)
 		(property "Value" "10k"
-			(at 66.04 107.9499 0)
+			(at 95.25 91.4401 0)
 			(effects
 				(font
@@
 		)
 		(property "Footprint" "Resistor_SMD:R_0603_1608Metric"
-			(at 61.722 106.68 90)
+			(at 99.568 92.71 90)
 			(effects
 				(font
@@
 		)
 		(property "Datasheet" "~"
-			(at 63.5 106.68 0)
+			(at 97.79 92.71 0)
 			(effects
 				(font
@@
 		)
 		(property "Description" "Resistor"
-			(at 63.5 106.68 0)
+			(at 97.79 92.71 0)
 			(effects
 				(font
@@
 		)
 		(property "Sim.Device" ""
-			(at 63.5 106.68 0)
+			(at 97.79 92.71 0)
 			(effects
 				(font
@@
 		)
 		(property "Sim.Pins" ""
-			(at 63.5 106.68 0)
+			(at 97.79 92.71 0)
 			(effects
 				(font
@@
 		)
 		(property "Sim.Type" ""
-			(at 63.5 106.68 0)
+			(at 97.79 92.71 0)
 			(effects
 				(font
@@
 	(symbol
 		(lib_id "Wall_E_parts:SI4435FDY-T1-GE3")
-		(at 63.5 95.25 0)
+		(at 93.98 104.14 180)
 		(unit 1)
 		(exclude_from_sim no)
@@
 		(fields_autoplaced yes)
 		(property "Reference" "Q1"
-			(at 78.74 87.63 0)
+			(at 78.74 88.9 0)
 			(effects
 				(font
@@
 		)
 		(property "Value" "SI4435FDY-T1-GE3"
-			(at 78.74 90.17 0)
+			(at 78.74 91.44 0)
 			(effects
 				(font
@@
 		)
 		(property "Footprint" "Wall_E_footprints:SO-8_VIS"
-			(at 63.5 95.25 0)
+			(at 93.98 104.14 0)
 			(effects
 				(font
@@
 		)
 		(property "Datasheet" "SI4435FDY-T1-GE3"
-			(at 63.5 95.25 0)
+			(at 93.98 104.14 0)
 			(effects
 				(font
@@
 		)
 		(property "Description" ""
-			(at 63.5 95.25 0)
+			(at 93.98 104.14 0)
 			(effects
 				(font
@@
 		)
 		(property "Sim.Device" ""
-			(at 63.5 95.25 0)
+			(at 93.98 104.14 0)
 			(effects
 				(font
@@
 		)
 		(property "Sim.Pins" ""
-			(at 63.5 95.25 0)
+			(at 93.98 104.14 0)
 			(effects
 				(font
@@
 		)
 		(property "Sim.Type" ""
-			(at 63.5 95.25 0)
-			(effects
-				(font
+			(at 93.98 104.14 0)
+			(effects
+				(font
